Commit message: changed initinal state

File: urdf/joystick.urdf (robot description, URDF)
Before this commit: robot joystick, 10 links, 9 joints
Links:
- added link pinch_bar_2; collision box size=0.05 0.02 0.002; visual box size=0.05 0.02 0.002
- link base_link: geometry collision box size=0.03 0.03 0.18; visual box size=0.03 0.03 0.18
- link pinch_bar_1: geometry collision box size=0.05 0.02 0.002; visual box size=0.05 0.02 0.002
- link pitch_bar_1: geometry collision cylinder length=0.13 radius=0.0125; visual cylinder length=0.13 radius=0.0125
- link pitch_bar_2: geometry collision box size=0.02 0.03 0.1; visual box size=0.02 0.03 0.1
- link pitch_bar_3: geometry collision box size=0.12 0.03 0.02; visual box size=0.12 0.03 0.02
- link roll_bar_1: geometry collision cylinder length=0.08 radius=0.0125; visual cylinder length=0.08 radius=0.0125
- link roll_bar_2: geometry collision cylinder length=0.07 radius=0.0065; visual cylinder length=0.07 radius=0.0065
- link yaw_bar_1: geometry collision cylinder length=0.075 radius=0.0125; visual cylinder length=0.075 radius=0.0125
- link yaw_bar_2: geometry collision box size=0.075 0.03 0.015; visual box size=0.075 0.03 0.015
- link yaw_bar_3: geometry collision box size=0.02 0.03 0.08; visual box size=0.02 0.03 0.08
Joints:
- added joint pinch2: type continuous, parent roll_bar_2, child pinch_bar_2, origin xyz=-0.07 0 -0.0065, axis 0 1 0, mimic joint=pinch multiplier=-1 offset=0
- joint pinch: axis 0 -1 0 -> 0 1 0; origin xyz=-0.07 0 0 -> xyz=-0.07 0 0.0065
- joint yaw_1: origin xyz=0 0 0.0175 -> xyz=0 0 0.0175 rpy=0 0 -1.570796

Commit message: colors changed

File: urdf/joystick.urdf (robot description, URDF)
Before this commit: robot joystick, 11 links, 10 joints
Links:
- added link base_pole; collision box size=0.03 0.03 0.18; visual box size=0.03 0.03 0.18
- link base_link: geometry visual box size=0.3 0.3 0.01
Joints:
- added joint base_: type fixed, parent base_link, child base_pole, origin xyz=0 0 0, axis 1 0 0
- joint pitch: parent base_link -> base_pole
